File: breakoutbrd.brd (EAGLE design)
At the start: 69.3 x 87 mm, 2 parts, among them U1 STM32F4XX

Commit message: update
Routing:
- net GND: track 97.5 -> 203.4 mm, vias 6 -> 3
- net CADDR1: track 55.5 -> 134.0 mm, vias 2 -> 5
- net VDD: track 63.4 -> 85.4 mm, vias 3 -> 1
- net CADDR3: track 85.1 -> 86.4 mm, vias 4 -> 5
- net CADDR0: track 57.3 -> 58.2 mm
- net CADDR11: track 81.9 -> 81.4 mm, vias 2 -> 0
- net CDATA2: track 41.7 -> 41.2 mm, vias 3 -> 2
- net CADDR12: vias 2 -> 0
- net CDATA0: vias 1 -> 3
- net CDATA6: vias 0 -> 1
- net CDATA5: vias 1 -> 0
- net CDATA3: vias 1 -> 0
- net CDATA1: vias 2 -> 0
- net CADDR9: vias 1 -> 0
- net CADDR7: vias 2 -> 1
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